File: hardware/kicad/parts-tally.kicad_sch (KiCad schematic)
At the start: 41 parts, among them J1 USB-C POWER ONLY, J2 LOAD CELL E+/E-/S+/S-, J3 UART DEBUG 3V3, SW1 TARE/CAL/RECOVERY, U1 Seeed XIAO ESP32-C3, U2 NAU7802SGI

Commit message: fix(hardware): resolve native KiCad ERC findings
Changed lines of the file:
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@@
-	)
-	(symbol
-		(lib_id "power:PWR_FLAG")
-		(at 284.48 54.61 0)
-		(unit 1)
-		(exclude_from_sim no)
-		(in_bom no)
-		(on_board yes)
-		(dnp no)
-		(fields_autoplaced no)
-		(property "Reference" "#FLG05"
-			(at 284.48 56.515 0.0000)
-			(effects
-				(font
-					(size 1.27 1.27)
-				)
-				(justify left)
-				(hide yes)
-			)
-		)
-		(property "Value" "PWR_FLAG"
-			(at 284.48 49.53 0)
-			(effects
-				(font
-					(size 1.27 1.27)
-				)
-			)
-		)
-		(property "Footprint" ""
-			(at 284.48 54.61 0.0000)
-			(effects
-				(font
-					(size 1.27 1.27)
-				)
-				(hide yes)
-			)
-		)
-		(property "Manufacturer" "N/A"
-			(at 287.02 59.6899 0)
-			(effects
-				(font
-					(size 1.27 1.27)
-				)
-				(justify left)
-			)
-		)
-		(property "MPN" "PCB_NET_FLAG"
-			(at 287.02 59.6899 0)
-			(effects
-				(font
-					(size 1.27 1.27)
-				)
-				(justify left)
-			)
-		)
-		(property "Supplier" "N/A"
-			(at 287.02 59.6899 0)
-			(effects
-				(font
-					(size 1.27 1.27)
-				)
-				(justify left)
-			)
-		)
-		(property "Supplier PN" "N/A"
-			(at 287.02 59.6899 0)
-			(effects
-				(font
-					(size 1.27 1.27)
-				)
-				(justify left)
-			)
-		)
-		(property "Datasheet" "~"
-			(at 284.48 54.61 0)
-			(effects
-				(font
-					(size 1.27 1.27)
-				)
-				(hide yes)
-			)
-		)
-		(property "Estimated Unit Cost USD" "0"
-			(at 287.02 59.6899 0)
-			(effects
-				(font
-					(size 1.27 1.27)
-				)
-				(justify left)
-			)
-		)
-		(property "Price Observed UTC" "2026-08-21"
-			(at 287.02 59.6899 0)
-			(effects
-				(font
-					(size 1.27 1.27)
-				)
-				(justify left)
-			)
-		)
-		(property "Stock Observed" "Not verified — distributor API credentials unavailable"
-			(at 287.02 59.6899 0)
-			(effects
-				(font
-					(size 1.27 1.27)
-				)
-				(justify left)
-			)
-		)
-		(property "Cost Basis" "Public distributor listing/search estimate; not a quote"
-			(at 287.02 59.6899 0)
-			(effects
-				(font
-					(size 1.27 1.27)
-				)
-				(justify left)
-			)
-		)
-		(property "BOM Comments" "ERC declaration only; not a physical BOM item."
-			(at 287.02 59.6899 0)
-			(effects
-				(font
-					(size 1.27 1.27)
-				)
-				(justify left)
-			)
-		)
-		(pin "1"
-		)
-		(instances
-			(project "Parts Tally carrier schematic"
-				(path "/efcb4a85-fdf6-4d70-bb67-1fd13c22d2fc"
-					(reference "#FLG05")
-					(unit 1)
-				)
-			)
-		)
 	)
 	(symbol
@@
 		)
 	)
-	(label "+3V3"
+	(label "GND"
 		(at 209.55 54.61 0.0000)
 		(effects
 			(font
-				(size 1.27 1.27)
-			)
-			(justify left bottom)
-		)
-	)
-	(label "AVDD_3V0"
-		(at 284.48 54.61 0.0000)
-		(effects
-			(font
